File: thermostat/thermostat.kicad_sch (KiCad schematic)
At the start: 14 parts, among them J1 Conn_01x16, J2 Conn_01x12, J3 Conn_01x05, SW1 EVP-AEBB2A, U1 ATSAMD21G18A-A, U2 SPX3819M5-L-3-3, U3 SS-52400-002, Y1 Crystal

Commit message: thermostat: Link symbols
Parts:
- SW1: symbol EVP-AEGE2A:EVP-AEBB2A -> SWITCH:EVP-AEBB2A
- U3: symbol SS-52400-002:SS-52400-002 -> USB:SS-52400-002
Changed lines of the file:
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@@
     (pin "1")
   )
-  (symbol (lib_id "EVP-AEGE2A:EVP-AEBB2A") (at 52.07 168.91 0) (unit 1)
+  (symbol (lib_id "SWITCH:EVP-AEBB2A") (at 52.07 168.91 0) (unit 1)
     (in_bom yes) (on_board yes) (fields_autoplaced)
     (property "Reference" "SW1" (id 0) (at 86.36 172.72 0)
@@
     (pin "2")
   )
-  (symbol (lib_id "SS-52400-002:SS-52400-002") (at 172.72 40.64 0) (unit 1)
+  (symbol (lib_id "USB:SS-52400-002") (at 172.72 40.64 0) (unit 1)
     (in_bom yes) (on_board yes) (fields_autoplaced)
     (property "Reference" "U3" (id 0) (at 198.12 25.4 0)
@@
       (effects (font (size 1.524 1.524)))
     )
-    (property "Footprint" "SS-52400-002_STW" (id 2) (at 198.12 33.02 0)
-      (effects (font (size 1.524 1.524)))
+    (property "Footprint" "SS-52400-002_STW" (id 2) (at 198.12 34.544 0)
+      (effects (font (size 1.524 1.524)) hide)
     )
     (property "Datasheet" "" (id 3) (at 172.72 40.64 0)
