File: esp32-ble-sensor-mini/150maPower.kicad_sch (KiCad schematic)
At the start: 3 parts, among them U5 TLV74333PDBVR

Commit message: esp32-c6-sensor v0.1 202507
Parts:
- U5: value TLV74333PDBVR -> TLV75533PDYDR
- renumbered C5 to C4
Connections:
- net GND: now also U5.4 (NR)
- net +5V renamed VIN
Changed lines of the file:
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@@
+	)
+	(junction
+		(at 125.73 92.71)
+		(diameter 0)
+		(color 0 0 0 0)
 	)
 	(junction
@@
 	(wire
 		(pts
+			(xy 133.35 85.09) (xy 133.35 92.71)
+		)
+		(stroke
+			(width 0)
+			(type default)
+		)
+	)
+	(wire
+		(pts
 			(xy 147.32 73.66) (xy 147.32 81.28)
 		)
@@
 		(pts
 			(xy 102.87 92.71) (xy 102.87 93.98)
+		)
+		(stroke
+			(width 0)
+			(type default)
+		)
+	)
+	(wire
+		(pts
+			(xy 125.73 92.71) (xy 133.35 92.71)
 		)
 		(stroke
@@
 		(on_board yes)
 		(dnp no)
-		(fields_autoplaced yes)
-		(property "Reference" "C5"
+		(property "Reference" "C4"
 			(at 140.97 92.7099 0)
 			(effects
@@
 			(project "esp32-ble-sensor"
 				(path "/f633b347-3747-472c-8d1d-c36902e3b057/5450845b-570e-422a-8597-439d9cbdf44b"
-					(reference "C5")
+					(reference "C4")
 					(unit 1)
 				)
@@
 			)
 		)
-		(property "Value" "TLV74333PDBVR"
+		(property "Value" "TLV75533PDYDR"
 			(at 125.73 78.74 0)
 			(effects
@@
 					(unit 1)
 				)
-			)
-		)
-	)
-	(symbol
-		(lib_id "power:+5V")
-		(at 102.87 78.74 0)
-		(unit 1)
-		(exclude_from_sim no)
-		(in_bom yes)
-		(on_board yes)
-		(dnp no)
-		(fields_autoplaced yes)
-		(property "Reference" "#PWR08"
-			(at 102.87 82.55 0)
-			(effects
-				(font
-					(size 1.27 1.27)
-				)
-				(hide yes)
-			)
-		)
-		(property "Value" "+5V"
-			(at 102.87 73.66 0)
-			(effects
-				(font
-					(size 1.27 1.27)
-				)
-			)
-		)
-		(property "Footprint" ""
-			(at 102.87 78.74 0)
-			(effects
-				(font
-					(size 1.27 1.27)
-				)
-				(hide yes)
-			)
-		)
-		(property "Datasheet" ""
-			(at 102.87 78.74 0)
-			(effects
-				(font
-					(size 1.27 1.27)
-				)
-				(hide yes)
-			)
-		)
-		(property "Description" "Power symbol creates a global label with name \"+5V\""
-			(at 102.87 78.74 0)
-			(effects
-				(font
-					(size 1.27 1.27)
-				)
-				(hide yes)
-			)
-		)
-		(pin "1"
-		)
-		(instances
-			(project "esp32-ble-sensor"
-				(path "/f633b347-3747-472c-8d1d-c36902e3b057/5450845b-570e-422a-8597-439d9cbdf44b"
-					(reference "#PWR08")
-					(unit 1)
-				)
