File: esp32-ble-sensor-mini/USBC2.0.kicad_sch (KiCad schematic)
At the start: 3 parts, among them J4 USB4215-03-A_REVA

Commit message: esp32-c6-sensor v0.1 202507
Parts:
- added U3: TPD4E05U06DQA, Package_SON:USON-10_2.5x1.0mm_P0.5mm, symbol Power_Protection:TPD4E05U06DQA
- R1, R2: footprint Resistor_SMD:R_1206_3216Metric -> Resistor_SMD:R_0603_1608Metric
Connections:
- net GND: now also U3.3 (GND), U3.8 (GND)
- net USB_D+: now also U3.1 (D1+), U3.10 (NC)
- net USB_D-: now also U3.2 (D1-), U3.9 (NC)
- net +5V renamed VBUS
- net VBUS: now also U3.5 (D2-), U3.6 (NC)
