File: esp32-ble-sensor-mini/_autosave-esp32-ble-sensor.kicad_sch (KiCad schematic)
At the start: 25 parts, among them J1 Conn_01x08_Pin, SW1 SW_SPST, SW2 SW_SPST, SW3 SW_SPST, U1 ESP32-C6-MINI-1/U, U4 SCD41-D-R2, U6 LM66200DRLR

Commit message: esp32-c6-sensor v0.1 202507
Connections:
- net VBAT_SENSE: now also U1.10 (MTDI/GPIO5/ADC1_CH5); no longer U1.19 (GPIO14)
Changed lines of the file:
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@@
+	(wire
+		(pts
+			(xy 68.58 81.28) (xy 83.82 81.28)
+		)
+		(stroke
+			(width 0)
+			(type default)
+		)
+	)
 	(wire
 		(pts
@@
 	(wire
 		(pts
+			(xy 83.82 81.28) (xy 83.82 82.55)
+		)
+		(stroke
+			(width 0)
+			(type default)
+		)
+	)
+	(wire
+		(pts
 			(xy 162.56 161.29) (xy 165.1 161.29)
 		)
@@
 		(pts
 			(xy 97.79 177.8) (xy 104.14 177.8)
-		)
-		(stroke
-			(width 0)
-			(type default)
-		)
-	)
-	(wire
-		(pts
-			(xy 83.82 81.28) (xy 83.82 82.55)
 		)
 		(stroke
@@
 		)
 	)
+	(label "VBAT_SENSE"
+		(at 68.58 81.28 180)
+		(effects
+			(font
+				(size 1.27 1.27)
+			)
+			(justify right bottom)
+		)
+	)
 	(label "SCL"
 		(at 101.6 29.21 0)
 		(effects
 			(font
-				(size 1.27 1.27)
-			)
-			(justify left bottom)
-		)
-	)
-	(label "VBAT_SENSE"
-		(at 152.4 97.79 0)
-		(effects
-			(font
