File: esp32-ble-sensor-mini/sht4x.kicad_sch (KiCad schematic)
At the start: 2 parts, among them U2 SHT4x

Commit message: esp32-c6-sensor v0.1 202507
Parts:
- C1: footprint Capacitor_SMD:C_1206_3216Metric -> Capacitor_SMD:C_0603_1608Metric
Changed lines of the file:
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@@
 			)
 		)
-		(property "Footprint" "Capacitor_SMD:C_1206_3216Metric"
+		(property "Footprint" "Capacitor_SMD:C_0603_1608Metric"
 			(at 158.4452 85.09 0)
 			(effects

Commit message: esp32 sensor 202509
Parts:
- renumbered C1 to C?, U2 to U?
Changed lines of the file:
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@@
 		(dnp no)
 		(fields_autoplaced yes)
-		(property "Reference" "C1"
+		(property "Reference" "C?"
 			(at 161.29 80.0099 0)
 			(effects
@@
 		)
 		(instances
+			(project "sht4x"
+				(path "/d7e596fe-744d-45f4-be6f-19b42f6fb9f0"
+					(reference "C?")
+					(unit 1)
+				)
+			)
 			(project "esp32-ble-sensor"
 				(path "/f633b347-3747-472c-8d1d-c36902e3b057/53c8d859-bbc4-4810-814c-ad11c4902857"
@@
 		(dnp no)
 		(fields_autoplaced yes)
-		(property "Reference" "#PWR05"
+		(property "Reference" "#PWR?"
 			(at 143.51 99.06 0)
 			(effects
@@
 		)
 		(instances
+			(project "sht4x"
+				(path "/d7e596fe-744d-45f4-be6f-19b42f6fb9f0"
+					(reference "#PWR?")
+					(unit 1)
+				)
+			)
 			(project "esp32-ble-sensor"
 				(path "/f633b347-3747-472c-8d1d-c36902e3b057/53c8d859-bbc4-4810-814c-ad11c4902857"
@@
 		(dnp no)
 		(fields_autoplaced yes)
-		(property "Reference" "#PWR06"
+		(property "Reference" "#PWR?"
 			(at 143.51 74.93 0)
 			(effects
@@
 		)
 		(instances
+			(project "sht4x"
+				(path "/d7e596fe-744d-45f4-be6f-19b42f6fb9f0"
+					(reference "#PWR?")
+					(unit 1)
+				)
+			)
 			(project "esp32-ble-sensor"
 				(path "/f633b347-3747-472c-8d1d-c36902e3b057/53c8d859-bbc4-4810-814c-ad11c4902857"
@@
 		(dnp no)
 		(fields_autoplaced yes)
-		(property "Reference" "U2"
+		(property "Reference" "U?"
 			(at 147.32 80.0099 0)
 			(effects
@@
 		)
 		(instances
+			(project "sht4x"
+				(path "/d7e596fe-744d-45f4-be6f-19b42f6fb9f0"
+					(reference "U?")
+					(unit 1)
+				)
+			)
 			(project "esp32-ble-sensor"
 				(path "/f633b347-3747-472c-8d1d-c36902e3b057/53c8d859-bbc4-4810-814c-ad11c4902857"
@@
 		)
 	)
+	(sheet_instances
+		(path "/"
+			(page "1")
+		)
+	)
+	(embedded_fonts no)
 )
